File: motherboard_pcb/2021_ver/buck_converters_v1.1.brd (EAGLE design)
At the start: 120.7 x 88.9 mm, 127 parts, among them J1 D15S24A4GV00LF, J4 171-025-213R001, Q1 IRFR5305, U2 TPS54302, U3 TPS54302, X5 332-02

Commit message: modified for silkscreen and 12V converter
Parts:
- renumbered U2 to U$2, U3 to U$3
Connections:
- net 12V: no longer J1.8
Routing:
- net 12V: track 97.0 -> 86.5 mm
Other:
- board text removed: "1"
- board text removed: "3V3"
- board text removed: "5"
- board text removed: "5V"
- board text removed: "6/12V"
- board text removed: "7"
- board text removed: "A"
- board text removed: "B_SCL"
- board text removed: "B_SDA"
- board text removed: "CANH"
- board text removed: "CANL"
- board text removed: "DROP_A"
- board text removed: "DROP_B"
- board text removed: "DROP_C"
- board text removed: "E"
- board text removed: "EN_5V"
- board text removed: "EN_6/12V"
- board text removed: "G"
- board text removed: "GND"
- board text removed: "Left Daughter Brd"
- board text removed: "M1_BK"
- board text removed: "M1_FR"
- board text removed: "M1_PG"
- board text removed: "M1_SV"
- board text removed: "M2_BK"
- board text removed: "M2_FR"
- board text removed: "M2_PG"
- board text removed: "M2_SV"
- board text removed: "M3_BK"
- board text removed: "M3_FR"
- board text removed: "M3_PG"
- board text removed: "M3_SV"
- board text removed: "M4_BK"
- board text removed: "M4_FR"
- board text removed: "M4_PG"
- board text removed: "M4_SV"
- board text removed: "M_EN"
- board text removed: "Motor"
- board text removed: "Motor Brd"
- board text removed: "NUSSEDS DARPASubT"
- board text removed: "Power Distribution Brd"
- board text removed: "Right Daughter Brd"
- board text removed: "Sensors, Comms"
- board text removed: "Sensors/Comms Brd"
- board text removed: "THER_A_SCL"
- board text removed: "THER_A_SDA"
- board text removed: "THER_B_SCL"
- board text removed: "THER_B_SDA"
- board text removed: "VER 1.1"
- board text removed: "VIN"
- board text removed: "VIN+"
- board text removed: "VIN-"
